File: Charger/Hardware/BoatBox/BoatBox.kicad_pcb (KiCad board)
At the start: 2 copper layers, 38 parts, among them Q201 IPD50R380CE, Q202 BSS138, Q301 IPD50R380CE, Q302 BSS138, Q401 IPD50R380CE, Q402 BSS138, Q501 IPD50R380CE, Q502 BSS138, X101 HCCPHPE24BKA90F, X102 HCCPHPE24BKA90F

Commit message: Layout update
Still in work
Parts:
- removed C201, C301, C401, C501: 10pF, Capacitor_SMD:C_0603_1608Metric_Pad1.05x0.95mm_HandSolder
- removed Q201, Q301, Q401, Q501: IPD50R380CE, Package_TO_SOT_SMD:TO-252-2
- removed Q202, Q302, Q402, Q502: BSS138, Package_TO_SOT_SMD:SOT-23
- removed R201, R301, R401, R501: 100R, Resistor_SMD:R_0603_1608Metric_Pad1.05x0.95mm_HandSolder
- removed R204, R304, R404, R504: 470k, Resistor_SMD:R_0603_1608Metric_Pad1.05x0.95mm_HandSolder
- removed X102: HCCPHPE24BKA90F, boatbox:HCCPHPE24BKA90F
- added C109: 100n, Capacitor_SMD:C_0603_1608Metric_Pad1.05x0.95mm_HandSolder, F.Cu at (76.7, 125.0)
- added C110: 100n, Capacitor_SMD:C_0603_1608Metric_Pad1.05x0.95mm_HandSolder, F.Cu at (92.1, 108.0)
- added C111: 10u, Capacitor_SMD:C_1210_3225Metric_Pad1.42x2.65mm_HandSolder, F.Cu at (74.2, 125.0)
- added C112: 270u, Capacitor_SMD:CP_Elec_10x10, F.Cu at (82.5, 106.0)
- added C113: 10u, Capacitor_SMD:C_1210_3225Metric_Pad1.42x2.65mm_HandSolder, F.Cu at (70.6, 125.0)
- added C114: 10u, Capacitor_SMD:C_1210_3225Metric_Pad1.42x2.65mm_HandSolder, F.Cu at (89.5, 108.6)
- added C115: 10u, Capacitor_SMD:C_1210_3225Metric_Pad1.42x2.65mm_HandSolder, F.Cu at (113.4, 128.9)
- added C116: 270u, Capacitor_SMD:CP_Elec_10x10, F.Cu at (82.5, 119.4)
- added C117: 68n, Capacitor_SMD:C_0603_1608Metric_Pad1.05x0.95mm_HandSolder, F.Cu at (83.1, 75.7)
- added C118: 68n, Capacitor_SMD:C_0603_1608Metric_Pad1.05x0.95mm_HandSolder, F.Cu at (98.3, 75.9)
- added C119: 68n, Capacitor_SMD:C_0603_1608Metric_Pad1.05x0.95mm_HandSolder, F.Cu at (113.3, 76.2)
- added C120: 68n, Capacitor_SMD:C_0603_1608Metric_Pad1.05x0.95mm_HandSolder, F.Cu at (128.4, 76.3)
- added C121: 270u, Capacitor_SMD:CP_Elec_10x10, F.Cu at (94.0, 119.4)
- added C122: 100n, Capacitor_SMD:C_0603_1608Metric_Pad1.05x0.95mm_HandSolder, F.Cu at (76.2, 118.1)
- added C124: 4.7n, Capacitor_SMD:C_0603_1608Metric, B.Cu at (50.3, 124.5)
- added C125: 4.7n, Capacitor_SMD:C_0603_1608Metric, B.Cu at (52.6, 103.4)
- added C126: 4.7n, Capacitor_SMD:C_0603_1608Metric, B.Cu at (52.7, 109.7)
- added C127: 4.7n, Capacitor_SMD:C_0603_1608Metric, B.Cu at (48.3, 100.8)
- added C128: 4.7n, Capacitor_SMD:C_0603_1608Metric, B.Cu at (61.5, 100.8)
- added C129: 4.7n, Capacitor_SMD:C_0603_1608Metric, B.Cu at (48.3, 104.4)
- added C130: 4.7n, Capacitor_SMD:C_0603_1608Metric, B.Cu at (61.5, 104.1)
- added C131: 4.7n, Capacitor_SMD:C_0603_1608Metric, B.Cu at (48.3, 111.0)
- added C132: 4.7n, Capacitor_SMD:C_0603_1608Metric, B.Cu at (61.5, 111.0)
- added C133: 4.7n, Capacitor_SMD:C_0603_1608Metric, B.Cu at (48.3, 107.7)
- added C134: 4.7n, Capacitor_SMD:C_0603_1608Metric, B.Cu at (61.5, 107.7)
- added D101: BAS16, Diode_SMD:D_SOT-23_ANK, F.Cu at (97.2, 131.4)
- added D102: BAS16, Diode_SMD:D_SOT-23_ANK, F.Cu at (107.3, 128.4)
- added D103: TL431D, Package_SO:SOIC-8_3.9x4.9mm_P1.27mm, F.Cu at (109.3, 121.3)
- added D105: MBRS360T3G, Diode_SMD:D_SMB_Handsoldering, F.Cu at (112.4, 138.0)
- added P101: TestPoint, TestPoint:TestPoint_Pad_D1.0mm, F.Cu at (89.5, 112.4)
- added P102: TestPoint, TestPoint:TestPoint_Pad_D1.0mm, F.Cu at (70.6, 129.3)
- added P103: TestPoint, TestPoint:TestPoint_Pad_D1.0mm, F.Cu at (73.9, 114.0)
- added P104: TestPoint, TestPoint:TestPoint_Pad_D1.0mm, F.Cu at (89.9, 104.1)
- added P105: TestPoint, TestPoint:TestPoint_Pad_D1.0mm, F.Cu at (69.1, 89.9)
- added P106: TestPoint, TestPoint:TestPoint_Pad_D1.0mm, F.Cu at (69.1, 91.7)
- added P107: TestPoint, TestPoint:TestPoint_Pad_D1.0mm, F.Cu at (69.1, 93.5)
- added P108: TestPoint, TestPoint:TestPoint_Pad_D1.0mm, F.Cu at (69.1, 95.2)
- added P109: TestPoint, TestPoint:TestPoint_Pad_D1.0mm, F.Cu at (113.3, 122.4)
- added P110: TestPoint, TestPoint:TestPoint_Pad_D1.0mm, F.Cu at (107.4, 114.6)
- added P111: TestPoint, TestPoint:TestPoint_Pad_D1.0mm, F.Cu at (118.6, 133.1)
- added P112: TestPoint, TestPoint:TestPoint_Pad_D1.0mm, F.Cu at (70.9, 119.6)
- added P113: TestPoint, TestPoint:TestPoint_Pad_D1.0mm, F.Cu at (84.8, 78.0)
- added P114: TestPoint, TestPoint:TestPoint_Pad_D1.0mm, F.Cu at (77.5, 89.9)
- added P115: TestPoint, TestPoint:TestPoint_Pad_D1.0mm, F.Cu at (99.8, 78.2)
- added P116: TestPoint, TestPoint:TestPoint_Pad_D1.0mm, F.Cu at (92.7, 90.2)
- added P117: TestPoint, TestPoint:TestPoint_Pad_D1.0mm, F.Cu at (114.8, 78.5)
- added P118: TestPoint, TestPoint:TestPoint_Pad_D1.0mm, F.Cu at (107.7, 90.4)
- added P119: TestPoint, TestPoint:TestPoint_Pad_D1.0mm, F.Cu at (130.0, 78.5)
- added P120: TestPoint, TestPoint:TestPoint_Pad_D1.0mm, F.Cu at (122.8, 90.6)
- added P201: TestPoint, TestPoint:TestPoint_Pad_D1.0mm, F.Cu at (73.0, 78.7)
- added P202: TestPoint, TestPoint:TestPoint_Pad_D1.0mm, F.Cu at (82.5, 85.7)
- added P301: TestPoint, TestPoint:TestPoint_Pad_D1.0mm, F.Cu at (88.3, 79.0)
- added P302: TestPoint, TestPoint:TestPoint_Pad_D1.0mm, F.Cu at (97.8, 86.0)
- added P401: TestPoint, TestPoint:TestPoint_Pad_D1.0mm, F.Cu at (103.3, 79.2)
- added P402: TestPoint, TestPoint:TestPoint_Pad_D1.0mm, F.Cu at (112.8, 86.2)
- added P501: TestPoint, TestPoint:TestPoint_Pad_D1.0mm, F.Cu at (118.1, 79.4)
- added P502: TestPoint, TestPoint:TestPoint_Pad_D1.0mm, F.Cu at (127.9, 86.4)
- added R101: 10k, Resistor_SMD:R_0603_1608Metric_Pad1.05x0.95mm_HandSolder, B.Cu at (73.7, 119.4)
- added R102: 46.4k, Resistor_SMD:R_0603_1608Metric_Pad1.05x0.95mm_HandSolder, F.Cu at (83.6, 73.2)
- added R103: 46.4k, Resistor_SMD:R_0603_1608Metric_Pad1.05x0.95mm_HandSolder, F.Cu at (98.8, 73.4)
- added R104: 46.4k, Resistor_SMD:R_0603_1608Metric_Pad1.05x0.95mm_HandSolder, F.Cu at (113.8, 73.7)
- added R105: 46.4k, Resistor_SMD:R_0603_1608Metric_Pad1.05x0.95mm_HandSolder, F.Cu at (128.9, 73.8)
- added R106: 46.4k, Resistor_SMD:R_0603_1608Metric_Pad1.05x0.95mm_HandSolder, B.Cu at (72.4, 121.9)
- added R107: 10k, Resistor_SMD:R_0603_1608Metric_Pad1.05x0.95mm_HandSolder, B.Cu at (77.7, 121.9)
- added R108: 46.4k, Resistor_SMD:R_0603_1608Metric_Pad1.05x0.95mm_HandSolder, F.Cu at (84.6, 75.7)
- added R109: 46.4k, Resistor_SMD:R_0603_1608Metric_Pad1.05x0.95mm_HandSolder, F.Cu at (99.8, 75.9)
- added R110: 46.4k, Resistor_SMD:R_0603_1608Metric_Pad1.05x0.95mm_HandSolder, F.Cu at (114.8, 76.2)
- added R111: 46.4k, Resistor_SMD:R_0603_1608Metric_Pad1.05x0.95mm_HandSolder, F.Cu at (129.9, 76.3)
- added R112: 1k, Resistor_SMD:R_0603_1608Metric_Pad1.05x0.95mm_HandSolder, F.Cu at (109.9, 128.9)
- added R114: 2.7R, Resistor_SMD:R_2816_7142Metric_Pad3.20x4.45mm_HandSolder, F.Cu at (112.9, 133.0)
- added R115: 1k, Resistor_SMD:R_0603_1608Metric_Pad1.05x0.95mm_HandSolder, F.Cu at (107.3, 125.9)
- added R116: 50m, Resistor_SMD:R_0603_1608Metric_Pad1.05x0.95mm_HandSolder, F.Cu at (110.9, 125.9)
- added R117: 10k, Potentiometer_THT:Potentiometer_Bourns_3296W_Vertical, F.Cu at (103.8, 116.7)
- added R118: 50m, Resistor_SMD:R_0603_1608Metric_Pad1.05x0.95mm_HandSolder, F.Cu at (108.5, 116.6)
- added R201A201: 1R, Resistor_SMD:R_1206_3216Metric_Pad1.42x1.75mm_HandSolder, F.Cu at (77.5, 74.9)
- added R201B201: 1R, Resistor_SMD:R_1206_3216Metric_Pad1.42x1.75mm_HandSolder, F.Cu at (74.9, 74.9)
- added R201C201: 1R, Resistor_SMD:R_1206_3216Metric_Pad1.42x1.75mm_HandSolder, F.Cu at (72.4, 74.9)
- added R301A301: 1R, Resistor_SMD:R_1206_3216Metric_Pad1.42x1.75mm_HandSolder, F.Cu at (92.7, 75.2)
- added R301B301: 1R, Resistor_SMD:R_1206_3216Metric_Pad1.42x1.75mm_HandSolder, F.Cu at (90.2, 75.2)
- added R301C301: 1R, Resistor_SMD:R_1206_3216Metric_Pad1.42x1.75mm_HandSolder, F.Cu at (87.6, 75.2)
- added R401A401: 1R, Resistor_SMD:R_1206_3216Metric_Pad1.42x1.75mm_HandSolder, F.Cu at (107.7, 75.4)
- added R401B401: 1R, Resistor_SMD:R_1206_3216Metric_Pad1.42x1.75mm_HandSolder, F.Cu at (105.2, 75.4)
- added R401C401: 1R, Resistor_SMD:R_1206_3216Metric_Pad1.42x1.75mm_HandSolder, F.Cu at (102.6, 75.4)
- added R501A501: 1R, Resistor_SMD:R_1206_3216Metric_Pad1.42x1.75mm_HandSolder, F.Cu at (120.2, 75.6)
- added R501B501: 1R, Resistor_SMD:R_1206_3216Metric_Pad1.42x1.75mm_HandSolder, F.Cu at (117.7, 75.6)
- added R501C501: 1R, Resistor_SMD:R_1206_3216Metric_Pad1.42x1.75mm_HandSolder, F.Cu at (122.8, 75.6)
- added S101: LM317, Package_TO_SOT_SMD:TO-252-2, F.Cu at (102.2, 130.2)
- added T101: IRFR5505PBF, Package_TO_SOT_SMD:TO-252-2, F.Cu at (77.5, 133.3)
- added T102: BSS138, Package_TO_SOT_SMD:SOT-23, B.Cu at (74.9, 121.9)
- added T103: IRFR5505PBF, Package_TO_SOT_SMD:TO-252-2, F.Cu at (85.1, 133.3)
- added T201: BC847, Package_TO_SOT_SMD:SOT-23, F.Cu at (80.6, 75.6)
- added T202: IPD50R380CE, Package_TO_SOT_SMD:TO-252-2, F.Cu at (77.5, 83.2)
- added T203: BSS138, Package_TO_SOT_SMD:SOT-23, F.Cu at (83.2, 79.4)
- added T301: BC847, Package_TO_SOT_SMD:SOT-23, F.Cu at (95.9, 75.8)
- added T302: IPD50R380CE, Package_TO_SOT_SMD:TO-252-2, F.Cu at (92.7, 83.4)
- added T303: BSS138, Package_TO_SOT_SMD:SOT-23, F.Cu at (98.4, 79.6)
- added T401: BC847, Package_TO_SOT_SMD:SOT-23, F.Cu at (110.9, 76.1)
- added T402: IPD50R380CE, Package_TO_SOT_SMD:TO-252-2, F.Cu at (107.7, 83.7)
- added T403: BSS138, Package_TO_SOT_SMD:SOT-23, F.Cu at (113.4, 79.9)
- added T501: BC847, Package_TO_SOT_SMD:SOT-23, F.Cu at (125.9, 76.2)
- added T502: IPD50R380CE, Package_TO_SOT_SMD:TO-252-2, F.Cu at (122.8, 83.8)
- added T503: BSS138, Package_TO_SOT_SMD:SOT-23, F.Cu at (128.5, 80.0)
- C101, C102, C103, C104, C105, C106, C107, C108: footprint Capacitor_SMD:C_0603_1608Metric_Pad1.05x0.95mm_HandSolder -> Capacitor_SMD:C_0603_1608Metric; moved to B.Cu
- R202, R302, R402, R502: value 10k -> 100k
- R203, R303, R403, R503: value 100k -> 470k
- moved C106 193.6 mm to (52.6, 114.3), turned to 90 degrees
- moved C102 192.4 mm to (54.6, 124.5), turned to 90 degrees
- moved C101 145.7 mm to (51.3, 94.2), turned to 180 degrees
- moved C108 141.5 mm to (48.3, 117.6), turned to 270 degrees
- moved C105 138.5 mm to (48.3, 114.3), turned to 90 degrees
- moved C107 133.9 mm to (52.6, 117.9), turned to 90 degrees
- moved C103 129.5 mm to (61.5, 96.8), turned to 180 degrees
- moved C104 128.9 mm to (61.5, 114.3), turned to 180 degrees
- moved X101 73.0 mm to (54.6, 109.2), turned to 270 degrees
- moved R303 59.7 mm to (98.4, 82.2)
- moved R302 56.2 mm to (98.4, 84.1), turned to 180 degrees
- moved R203 53.6 mm to (83.2, 81.9), turned to 0 degrees
- moved R502 52.8 mm to (128.5, 84.5), turned to 180 degrees
- moved R402 46.7 mm to (113.4, 84.3), turned to 180 degrees
- moved R202 46.0 mm to (83.2, 83.8), turned to 180 degrees
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Connections:
- C101 pad 2: /A_S_DIAG1 -> UBD
- C102 pad 2: /A_T_OUT1 -> UBD
- C103 pad 2: /A_S_DIAG2 -> /E_S_RLY
- C104 pad 2: /A_T_OUT2 -> /U_U_CHRG
- C105 pad 2: /A_S_DIAG3 -> /E_S_CTL1
- C106 pad 2: /A_T_OUT3 -> /E_S_CTL2
- C107 pad 2: /A_S_DIAG4 -> /E_S_CTL3
- C108 pad 2: /A_T_OUT4 -> /E_S_CTL4
- R202 pad 1: Net-(C201-Pad1) -> /A_T_OUT1
- R202 pad 2: GND -> Net-(P202-Pad1)
- R203 pad 1: /A_T_OUT1 -> Net-(P202-Pad1)
- R203 pad 2: Net-(Q202-Pad1) -> GND
- R302 pad 1: Net-(C301-Pad1) -> /A_T_OUT2
- R302 pad 2: GND -> Net-(P302-Pad1)
- R303 pad 1: /A_T_OUT2 -> Net-(P302-Pad1)
- R303 pad 2: Net-(Q302-Pad1) -> GND
- R402 pad 1: Net-(C401-Pad1) -> /A_T_OUT3
- R402 pad 2: GND -> Net-(P402-Pad1)
- R403 pad 1: /A_T_OUT3 -> Net-(P402-Pad1)
- R403 pad 2: Net-(Q402-Pad1) -> GND
- R502 pad 1: Net-(C501-Pad1) -> /A_T_OUT4
- R502 pad 2: GND -> Net-(P502-Pad1)
- R503 pad 1: /A_T_OUT4 -> Net-(P502-Pad1)
- R503 pad 2: Net-(Q502-Pad1) -> GND
- X101 pad 1: GND -> UBD
- X101 pad 10: Net-(X101-Pad10) -> UBR
- X101 pad 11: Net-(X101-Pad11) -> UBR
- X101 pad 12: Net-(X101-Pad12) -> UBR
- X101 pad 13: Net-(X101-Pad13) -> UBR
- X101 pad 14: Net-(X101-Pad14) -> /E_S_CTL2
- X101 pad 15: Net-(X101-Pad15) -> /E_S_CTL3
- X101 pad 16: Net-(X101-Pad16) -> UBD
- X101 pad 17: Net-(X101-Pad17) -> /E_S_RLY
- X101 pad 18: /A_S_DIAG1 -> /A_T_OUT1
- X101 pad 19: /A_T_OUT1 -> /A_T_OUT2
- X101 pad 2: GND -> /A_S_DIAG1
- X101 pad 20: /A_S_DIAG2 -> /A_T_OUT3
- X101 pad 21: /A_T_OUT2 -> /A_T_OUT4
- X101 pad 22: /A_S_DIAG3 -> /U_U_CHRG
- X101 pad 23: /A_T_OUT3 -> GND
- X101 pad 24: /A_S_DIAG4 -> GND
- X101 pad 3: GND -> /A_S_DIAG2
- X101 pad 4: Net-(X101-Pad4) -> /A_S_DIAG3
- X101 pad 5: Net-(X101-Pad5) -> /A_S_DIAG4
- X101 pad 6: Net-(X101-Pad6) -> /E_S_CTL1
- X101 pad 7: Net-(X101-Pad7) -> /E_S_CTL4
- X101 pad 8: Net-(X101-Pad8) -> UBR
- X101 pad 9: Net-(X101-Pad9) -> GND
Routing:
- net /E_S_CTL4: track 0.00 -> 128.8 mm, vias 0 -> 4
- net UBD: track 0.00 -> 121.1 mm, vias 0 -> 1
- net /E_S_CTL3: track 0.00 -> 114.8 mm, vias 0 -> 2
- net /A_S_DIAG4: track 0.00 -> 110.5 mm, vias 0 -> 1
- net /E_S_CTL2: track 0.00 -> 106.9 mm, vias 0 -> 2
- net /A_S_DIAG3: track 0.00 -> 93.1 mm, vias 0 -> 1
- net /A_T_OUT4: track 0.00 -> 89.3 mm
- net /E_S_CTL1: track 0.00 -> 87.9 mm, vias 0 -> 3
- net UBR: track 0.00 -> 84.7 mm
- net /A_S_DIAG2: track 0.00 -> 75.3 mm, vias 0 -> 1
- net /U_U_CHRG: track 0.00 -> 73.6 mm
- net /A_T_OUT3: track 0.00 -> 72.8 mm
- net /A_S_DIAG1: track 0.00 -> 56.2 mm, vias 0 -> 1
- net /A_T_OUT2: track 0.00 -> 56.0 mm
- net GND: track 10.9 -> 64.8 mm, vias 0 -> 30
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- added copper zone on F.Cu, net /U_U_CHRG
- added copper zone on B.Cu, net GND
- added copper zone on F.Cu, net GND
- added copper zone on F.Cu, net Net-(C115-Pad1)
- added copper zone on F.Cu, net Net-(D105-Pad2)
- added copper zone on F.Cu, net Net-(P201-Pad1)
- added copper zone on F.Cu, net Net-(P301-Pad1)
- added copper zone on F.Cu, net Net-(P401-Pad1)
- added copper zone on F.Cu, net Net-(P501-Pad1)
- added copper zone on F.Cu, net Net-(T101-Pad2)
- added copper zone on F.Cu, net UBD
- added copper zone on F.Cu, net UBR

Commit message: WIP commit
squash after finish.
Parts:
- added ?: , boatbox:Zeichnung, F.Cu at (293.4, 149.0)
- added REF**: MountingHole_4mm, MountingHole:MountingHole_4mm, F.Cu at (237.9, 150.0)
- added REF**: BUMP-SR0.8-3.0, boatbox:BUMP-SR0.8-3.0, B.Cu at (218.9, 72.5)
- added REF**: BUMP-SR0.8-3.0, boatbox:BUMP-SR0.8-3.0, B.Cu at (211.0, 77.0)
- added REF**: BUMP-SR0.8-3.0, boatbox:BUMP-SR0.8-3.0, B.Cu at (205.1, 77.0)
- added REF**: BUMP-SR0.8-3.0, boatbox:BUMP-SR0.8-3.0, B.Cu at (197.0, 77.0)
- added REF**: BUMP-SR0.8-3.0, boatbox:BUMP-SR0.8-3.0, B.Cu at (184.8, 77.1)
- added REF**: MountingHole_4mm, MountingHole:MountingHole_4mm, F.Cu at (234.9, 69.1)
- added REF**: MountingHole_4mm, MountingHole:MountingHole_4mm, F.Cu at (165.0, 69.1)
- added REF**: MountingHole_4mm, MountingHole:MountingHole_4mm, F.Cu at (165.0, 150.0)
- added REF**: BUMP-SR0.8-3.0, boatbox:BUMP-SR0.8-3.0, B.Cu at (223.7, 82.4)
- added REF**: BUMP-SR0.8-3.0, boatbox:BUMP-SR0.8-3.0, B.Cu at (213.3, 83.2)
- added REF**: BUMP-SR0.8-3.0, boatbox:BUMP-SR0.8-3.0, B.Cu at (189.4, 82.4)
- added REF**: BUMP-SR0.8-3.0, boatbox:BUMP-SR0.8-3.0, B.Cu at (192.9, 77.1)
- added REF**: BUMP-SR0.8-3.0, boatbox:BUMP-SR0.8-3.0, B.Cu at (226.7, 77.0)
- D103: value TL431D -> NCP431; footprint Package_SO:SOIC-8_3.9x4.9mm_P1.27mm -> Package_TO_SOT_SMD:SOT-23
- D105: footprint Diode_SMD:D_SMB_Handsoldering -> Diode_SMD:D_SMC_Handsoldering
- R101, R106, R107, T102: moved to F.Cu
- R117: footprint Potentiometer_THT:Potentiometer_Bourns_3296W_Vertical -> boatbox:Potentiometer_Cemet_23A_Horizontal
- moved C124 202.7 mm to (250.8, 94.3), turned to 270 degrees
- moved C108 200.3 mm to (248.6, 114.8), turned to 90 degrees
- moved C133 200.3 mm to (248.6, 108.2)
- moved C127 200.3 mm to (248.6, 101.2)
- moved C131 200.3 mm to (248.6, 111.3)
- moved C129 200.3 mm to (248.6, 104.3)
- moved C125 200.1 mm to (252.6, 108.6), turned to 270 degrees
- moved C126 200.0 mm to (252.6, 103.8)
- moved C101 199.5 mm to (248.6, 124.3), turned to 0 degrees
- moved C105 196.2 mm to (244.4, 117.9), turned to 270 degrees
- moved C107 196.0 mm to (248.6, 117.9), turned to 270 degrees
- moved C102 194.2 mm to (246.4, 94.1), turned to 270 degrees
- moved X101 191.9 mm to (246.5, 109.5), turned to 90 degrees
- moved C106 191.8 mm to (244.4, 114.8)
- moved C134 182.9 mm to (244.4, 108.2), turned to 90 degrees
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Connections:
- D103 pad 1: Net-(D102-Pad1) -> Net-(D103-Pad1)
- D103 pad 2: GND -> Net-(D102-Pad1)
- P110 pad 1: Net-(D103-Pad8) -> Net-(D103-Pad1)
- R117 pad 2: Net-(D103-Pad8) -> Net-(D103-Pad1)
- X101 pad 10: UBR -> /E_S_CTL1
- X101 pad 11: UBR -> /E_S_CTL2
- X101 pad 12: UBR -> /A_S_DIAG4
- X101 pad 13: UBR -> /A_S_DIAG3
- X101 pad 14: /E_S_CTL2 -> /A_S_DIAG2
- X101 pad 15: /E_S_CTL3 -> /A_S_DIAG1
- X101 pad 17: /E_S_RLY -> GND
- X101 pad 18: /A_T_OUT1 -> /U_U_CHRG
- X101 pad 19: /A_T_OUT2 -> /E_S_RLY
- X101 pad 2: /A_S_DIAG1 -> /E_S_CTL3
- X101 pad 20: /A_T_OUT3 -> /A_T_OUT4
- X101 pad 21: /A_T_OUT4 -> /A_T_OUT3
- X101 pad 22: /U_U_CHRG -> /A_T_OUT2
- X101 pad 23: GND -> /A_T_OUT1
- X101 pad 3: /A_S_DIAG2 -> /E_S_CTL4
- X101 pad 4: /A_S_DIAG3 -> UBR
- X101 pad 5: /A_S_DIAG4 -> UBR
- X101 pad 6: /E_S_CTL1 -> UBR
- X101 pad 7: /E_S_CTL4 -> UBR
Routing:
- net /E_S_CTL4: track 128.8 -> 32.2 mm, vias 4 -> 0
- net /E_S_CTL3: track 114.8 -> 28.8 mm, vias 2 -> 0
- net /E_S_CTL2: track 106.9 -> 26.0 mm, vias 2 -> 0
- net GND: track 64.8 -> 133.3 mm, vias 30 -> 152
- net /E_S_CTL1: track 87.9 -> 22.1 mm, vias 3 -> 0
- net /LSS 3/ctrl: track 8.82 -> 54.7 mm, vias 0 -> 2
- net /LSS 4/ctrl: track 8.86 -> 54.7 mm
- net /LSS 2/ctrl: track 8.82 -> 45.4 mm, vias 0 -> 2
- net /A_S_DIAG3: track 93.1 -> 64.2 mm, vias 1 -> 0
- net UBD: track 121.1 -> 93.7 mm, vias 1 -> 17
- net /LSS 1/ctrl: track 8.82 -> 35.8 mm, vias 0 -> 2
- net /A_S_DIAG1: track 56.2 -> 36.6 mm, vias 1 -> 0
- net /A_S_DIAG4: track 110.5 -> 93.7 mm, vias 1 -> 2
- net Net-(R116-Pad2): track 16.8 -> 2.36 mm, vias 1 -> 0
- net UBR: track 84.7 -> 70.3 mm, vias 0 -> 3
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- added copper zone on B.Cu, net /A_T_OUT1
- added copper zone on B.Cu, net /A_T_OUT2
- added copper zone on B.Cu, net /A_T_OUT3
- added copper zone on B.Cu, net /A_T_OUT4
- added copper zone on B.Cu, net Net-(C115-Pad1)
- added copper zone on B.Cu, net Net-(P201-Pad1)
- added copper zone on B.Cu, net Net-(P301-Pad1)
- added copper zone on B.Cu, net Net-(P401-Pad1)
- added copper zone on B.Cu, net Net-(P501-Pad1)
- added copper zone on B.Cu, net Net-(T101-Pad2)
- added copper zone on B.Cu, net UBD
Other:
- board outline added: 97.2 x 86.3 mm
- net class 3A added: clearance 0.3, trace_width 1, via_dia 1.6, via_drill 0.8
- net class 6A added: clearance 0.3, trace_width 2, via_dia 1.6, via_drill 0.8

Commit message: WIP
Parts:
- removed R501B501: 1R, Resistor_SMD:R_1206_3216Metric_Pad1.42x1.75mm_HandSolder
- added R501B: 1R, Resistor_SMD:R_1206_3216Metric_Pad1.42x1.75mm_HandSolder, F.Cu at (194.2, 87.3)
- added REF**: BUMP-SR0.8-3.0, boatbox:BUMP-SR0.8-3.0, B.Cu at (201.4, 72.1)
- added REF**: BUMP-SR0.8-3.0, boatbox:BUMP-SR0.8-3.0, B.Cu at (188.6, 141.3)
- added REF**: BUMP-SR0.8-3.0, boatbox:BUMP-SR0.8-3.0, B.Cu at (192.8, 145.8)
- added REF**: BUMP-SR0.8-3.0, boatbox:BUMP-SR0.8-3.0, B.Cu at (205.4, 138.8)
- added REF**: BUMP-SR0.8-3.0, boatbox:BUMP-SR0.8-3.0, B.Cu at (224.7, 88.7)
- added REF**: BUMP-SR0.8-3.0, boatbox:BUMP-SR0.8-3.0, B.Cu at (228.2, 88.7)
- added REF**: BUMP-SR0.8-3.0, boatbox:BUMP-SR0.8-3.0, B.Cu at (213.2, 89.0)
- added REF**: BUMP-SR0.8-3.0, boatbox:BUMP-SR0.8-3.0, B.Cu at (216.8, 89.0)
- added REF**: BUMP-SR0.8-3.0, boatbox:BUMP-SR0.8-3.0, B.Cu at (204.9, 88.7)
- added REF**: BUMP-SR0.8-3.0, boatbox:BUMP-SR0.8-3.0, B.Cu at (201.3, 88.7)
- added REF**: BUMP-SR0.8-3.0, boatbox:BUMP-SR0.8-3.0, B.Cu at (193.7, 88.7)
- added REF**: BUMP-SR0.8-3.0, boatbox:BUMP-SR0.8-3.0, B.Cu at (189.0, 72.2)
- added REF**: BUMP-SR0.8-3.0, boatbox:BUMP-SR0.8-3.0, B.Cu at (190.1, 88.7)
- added REF**: BUMP-SR0.8-3.0, boatbox:BUMP-SR0.8-3.0, B.Cu at (199.3, 133.7)
- added REF**: BUMP-SR0.8-3.0, boatbox:BUMP-SR0.8-3.0, B.Cu at (199.3, 144.9)
- added REF**: BUMP-SR0.8-3.0, boatbox:BUMP-SR0.8-3.0, B.Cu at (212.5, 146.1)
- added REF**: BUMP-SR0.8-3.0, boatbox:BUMP-SR0.8-3.0, B.Cu at (212.5, 128.9)
- added REF**: BUMP-SR0.8-3.0, boatbox:BUMP-SR0.8-3.0, B.Cu at (208.4, 132.8)
- added REF**: BUMP-SR0.8-3.0, boatbox:BUMP-SR0.8-3.0, B.Cu at (217.2, 139.8)
- added REF**: BUMP-SR0.8-3.0, boatbox:BUMP-SR0.8-3.0, B.Cu at (217.2, 132.7)
- renumbered R201A201 to R201A, R201B201 to R201B, R201C201 to R201C, R301A301 to R301A, R301B301 to R301B, R301C301 to R301C, R401A401 to R401A, R401B401 to R401B, R401C401 to R401C, R501A501 to R501A, R501C501 to R501C
Routing:
- net UBD: track 93.7 -> 120.2 mm
- net Net-(R106-Pad2): track 0.00 -> 5.29 mm
- net Net-(R107-Pad1): track 12.3 -> 17.3 mm
- net Net-(C115-Pad1): track 15.8 -> 19.1 mm
- net /E_S_RLY: track 40.0 -> 38.7 mm
- net GND: track 133.3 -> 134.5 mm, vias 152 -> 198
- net /LSS 1/ctrl: track 35.8 -> 36.6 mm
- added copper zone on B.Cu, net Net-(D105-Pad2)
